Commit message: urdf tutorials

File: urdf/tutorial1.urdf (robot description, URDF)
Before this commit: robot firstbot, 1 links, 0 joints
Links:
- added link box; visual box size=0.08 0.08 0.08
- added link gripper_pole; visual cylinder length=0.2 radius=0.01
- added link head; visual sphere radius=0.2
- added link left_gripper; visual mesh filename=package://urdf_tutorial/meshes/l_finger.dae
- added link left_leg; visual box size=0.6 0.1 0.2
- added link left_tip; visual mesh filename=package://urdf_tutorial/meshes/l_finger_tip.dae
- added link right_base; visual box size=0.4 0.1 0.1
- added link right_front_wheel; visual cylinder length=0.1 radius=0.035
- added link right_leg; visual box size=0.6 0.1 0.2
Joints:
- added joint base_to_left_leg: type fixed, parent base_link, child left_leg, origin xyz=0 0.22 0.25
- added joint base_to_right_leg: type fixed, parent base_link, child right_leg, origin xyz=0 -0.22 0.25
- added joint gripper_extension: type fixed, parent base_link, child gripper_pole, origin xyz=0.19 0 0.2 rpy=0 0 0
- added joint head_swivel: type fixed, parent base_link, child head, origin xyz=0 0 0.3
- added joint left_gripper_joint: type fixed, parent gripper_pole, child left_gripper, origin xyz=0.2 0.01 0
- added joint left_tip_joint: type fixed, parent left_gripper, child left_tip
- added joint right_base_joint: type fixed, parent right_leg, child right_base, origin xyz=0 0 -0.6
- added joint right_front_wheel_joint: type fixed, parent right_base, child right_front_wheel, origin xyz=0.13333 0 -0.085
- added joint tobox: type fixed, parent head, child box, origin xyz=0.1814 0 0.1414
