Commit message: style and pose fix

File: models/panda.srdf.xacro (robot description, xacro)
@@ -17,4 +17,8 @@
     <group name="panda_arm" />
     <group name="hand" />
+  </group>
+  <group name="panda_arm_hand_table">
+    <group name="panda_arm_hand"/>
+    <group name="base_link"/>
   </group>
   <group_state name="open" group="hand">
@@ -41,5 +45,15 @@
   <disable_collisions link1="panda_link7" link2="panda_rightfinger" reason="Never" />
   <disable_collisions link1="panda_link8" link2="panda_rightfinger" reason="Never" />
-  <disable_collisions link1="panda_link0" link2="base_link" reason="Adjacent"/>
+  <disable_collisions link1="panda_link0" link2="base" reason="Adjacent"/>
   <disable_collisions link1="panda_link1" link2="base_link" reason="Adjacent"/>
+  <disable_collisions link1="panda_link2" link2="base_link" reason="Adjacent"/>
+  <disable_collisions link1="panda_link3" link2="base_link" reason="Adjacent"/>
+  <disable_collisions link1="panda_link4" link2="base_link" reason="Adjacent"/>
+  <disable_collisions link1="panda_link5" link2="base_link" reason="Adjacent"/>
+  <disable_collisions link1="panda_link6" link2="base_link" reason="Adjacent"/>
+  <disable_collisions link1="panda_link7" link2="base_link" reason="Adjacent"/>
+  <disable_collisions link1="panda_link8" link2="base_link" reason="Adjacent"/>
+  <disable_collisions link1="panda_hand" link2="base_link" reason="Adjacent"/>
+  <disable_collisions link1="panda_leftfinger" link2="base_link" reason="Adjacent"/>
+  <disable_collisions link1="panda_rightfinger" link2="base_link" reason="Adjacent"/>
 </robot>

File: models/panda.urdf (robot description, URDF)
Before this commit: robot panda, 1 links, 1 joints
Links:
- link base_link: geometry collision cylinder length=1 radius=1; collision mesh filename=package://jgioia_panda_projects/models/table_collision.STL scale=0.001 0.001 0.001

Commit message: better model

File: models/panda.srdf.xacro (robot description, xacro)
@@ -46,14 +46,3 @@
   <disable_collisions link1="panda_link8" link2="panda_rightfinger" reason="Never" />
   <disable_collisions link1="panda_link0" link2="base_link" reason="Adjacent"/>
-  <disable_collisions link1="panda_link1" link2="base_link" reason="Adjacent"/>
-  <disable_collisions link1="panda_link2" link2="base_link" reason="Adjacent"/>
-  <disable_collisions link1="panda_link3" link2="base_link" reason="Adjacent"/>
-  <disable_collisions link1="panda_link4" link2="base_link" reason="Adjacent"/>
-  <disable_collisions link1="panda_link5" link2="base_link" reason="Adjacent"/>
-  <disable_collisions link1="panda_link6" link2="base_link" reason="Adjacent"/>
-  <disable_collisions link1="panda_link7" link2="base_link" reason="Adjacent"/>
-  <disable_collisions link1="panda_link8" link2="base_link" reason="Adjacent"/>
-  <disable_collisions link1="panda_hand" link2="base_link" reason="Adjacent"/>
-  <disable_collisions link1="panda_leftfinger" link2="base_link" reason="Adjacent"/>
-  <disable_collisions link1="panda_rightfinger" link2="base_link" reason="Adjacent"/>
 </robot>

File: models/panda.urdf (robot description, URDF)
Before this commit: robot panda, 2 links, 2 joints
Links:
- link base_link: geometry collision mesh filename=package://jgioia_panda_projects/models/table.STL scale=0.001 0.001 0.001; visual mesh filename=package://jgioia_panda_projects/models/table.STL scale=0.001 0.001 0.001
