Commit message: model fix

File: models/panda.urdf (robot description, URDF)
Before this commit: robot panda, 1 links, 1 joints
Links:
- link base_link: geometry collision cylinder length=1 radius=1; visual mesh filename=package://jgioia_panda_projects/models/table.STL scale=0.001 0.001 0.001

Commit message: this stuff is broken

File: models/panda.urdf (robot description, URDF)
Before this commit: robot panda, 1 links, 1 joints
Links:
- added link world
Joints:
- removed joint table_robot_joint
- added joint table_world_joint: type fixed, parent base_link, child world, origin xyz=0 0 0 rpy=0 0 -1.57075
- added joint world_panda_joint: type fixed, parent world, child panda_link0, origin xyz=0 0 0 rpy=0 0 0

Commit message: camera and other refractoring

File: models/panda.urdf (robot description, URDF)
Before this commit: robot panda, 2 links, 2 joints
Links:
- removed link base_link
- removed link world
Joints:
- removed joint table_world_joint
- removed joint world_panda_joint
