Commit message: demos are close

File: models/box_purple.xacro (robot description, xacro)
@@ -1,12 +1,4 @@
 <?xml version="1.0"?>
 <robot xmlns:xacro="http://www.ros.org/wiki/xacro" name="simple_box">
-    <!-- <link name="object_base_link">
-    </link>
-    <joint name="object_base_joint" type="fixed">
-        <parent link="object_base_link"/>
-        <child link="object_link"/>
-        <axis xyz="0 0 1" />
-        <origin xyz="0.4 -0.5 0.4" rpy="0 0 0"/>
-    </joint> -->
     <link name="object_link">
         <origin xyz="0.4 -0.5 0.4" />
@@ -28,6 +20,6 @@
     <gazebo reference="object_link">
         <material>Gazebo/Purple</material>
-        <mu1>100</mu1>
-        <mu2>100</mu2>
+        <mu1>0.2</mu1>
+        <mu2>0.2</mu2>
         <gravity>1</gravity>
     </gazebo>

Commit message: cleanup

File: models/box_purple.xacro (robot description, xacro)
@@ -1,3 +1,4 @@
 <?xml version="1.0"?>
+<!-- A purple 0.03x0.03x0.03 box.-->
 <robot xmlns:xacro="http://www.ros.org/wiki/xacro" name="simple_box">
     <link name="object_link">

File: models/box_yellow.xacro (robot description, xacro)
@@ -1,3 +1,4 @@
 <?xml version="1.0"?>
+<!-- A yellow 0.03x0.03x0.03 box.-->
 <robot xmlns:xacro="http://www.ros.org/wiki/xacro" name="simple_box">
     <link name="object_link">

File: models/panda_table.srdf.xacro (robot description, xacro)
@@ -1,7 +1,4 @@
 <?xml version='1.0' encoding='utf-8'?>
-<!--This does not replace URDF, and is not an extension of URDF.
-    This is a format for representing semantic information about the robot structure.
-    A URDF file must exist for this robot as well, where the joints and the links that are referenced are defined
--->
+<!-- Semantic description for the model of the panda + table. -->
 <robot xmlns:xacro="http://www.ros.org/wiki/xacro" name="panda">
   <xacro:include filename="$(find moveit_resources_panda_moveit_config)/config/panda_arm.xacro" />
@@ -20,5 +17,5 @@
   <group name="panda_arm_hand_table">
     <group name="panda_arm_hand"/>
-    <group name="base_link"/>
+    <group name="table"/>
   </group>
   <group_state name="open" group="hand">
@@ -45,4 +42,4 @@
   <disable_collisions link1="panda_link7" link2="panda_rightfinger" reason="Never" />
   <disable_collisions link1="panda_link8" link2="panda_rightfinger" reason="Never" />
-  <disable_collisions link1="panda_link0" link2="base_link" reason="Adjacent"/>
+  <disable_collisions link1="panda_link0" link2="table" reason="Adjacent"/>
 </robot>

File: models/panda_table.urdf (robot description, URDF)
Before this commit: robot panda, 2 links, 2 joints
Links:
- removed link world
- added link table; collision mesh filename=package://jgioia_panda_projects/models/table.STL scale=0.001 0.001 0.001; visual mesh filename=package://jgioia_panda_projects/models/table.STL scale=0.001 0.001 0.001
- link base_link: geometry 
Joints:
- removed joint table_world_joint
- added joint world_table_joint: type fixed, parent base_link, child table, origin xyz=0 0 0 rpy=0 0 1.57075
- joint world_panda_joint: parent world -> base_link
